Commit message: Fix can problems and services

File: urdf/powerball_gripper_bak.urdf (robot description, URDF)
Before this commit: robot powerball, 14 links, 13 joints
Joints:
- joint arm_0_joint: origin xyz=0 0 0.14 rpy=0 0 0 -> xyz=0 0 0.5 rpy=3.1415926 0 0
- joint arm_1_joint: origin xyz=0 0 0.0897 rpy=0 0 0 -> xyz=0 0 -0.0897 rpy=0 0 0
- joint arm_2_joint: origin xyz=0 0 0 rpy=-1.5708 0 3.14159 -> xyz=0 0 0 rpy=1.5708 0 0
